Commit message: Rebase from 'upstream'

File: ffw_description/ros2_control/ffw_bg2_rev4_follower/ffw_bg2_follower.ros2_control.xacro (robot description, xacro)
@@ -2,6 +2,5 @@
 <robot xmlns:xacro="http://www.ros.org/wiki/xacro">
   <xacro:macro name="ffw_bg2_follower_system" params="use_sim:=^|false use_fake_hardware:=^|false fake_sensor_commands:=^|false">
-    <xacro:property name="initial_positions" value="${load_yaml(initial_positions_file)['initial_positions']}"/>
-    <ros2_control name="ffw_bg2_follower" type="system">
+    <ros2_control name="ffw_bg2_follower" type="system" is_async="true">
       <xacro:if value="$(arg use_sim)">
         <hardware>
@@ -23,4 +22,5 @@
             <param name="number_of_joints">19</param>
             <param name="number_of_transmissions">19</param>
+            <param name="disable_torque_at_init">true</param>
             <param name="transmission_to_joint_matrix">
               1, 0, 0, 0, 0, 0, 0, 0, 0, 0, 0, 0, 0, 0, 0, 0, 0, 0, 0,
@@ -77,4 +77,5 @@
         <state_interface name="position"/>
         <state_interface name="velocity"/>
+        <state_interface name="effort"/>
       </joint>
       <joint name="arm_r_joint2">
@@ -82,4 +83,5 @@
         <state_interface name="position"/>
         <state_interface name="velocity"/>
+        <state_interface name="effort"/>
       </joint>
       <joint name="arm_r_joint3">
@@ -87,4 +89,5 @@
         <state_interface name="position"/>
         <state_interface name="velocity"/>
+        <state_interface name="effort"/>
       </joint>
       <joint name="arm_r_joint4">
@@ -92,4 +95,5 @@
         <state_interface name="position"/>
         <state_interface name="velocity"/>
+        <state_interface name="effort"/>
       </joint>
       <joint name="arm_r_joint5">
@@ -97,4 +101,5 @@
         <state_interface name="position"/>
         <state_interface name="velocity"/>
+        <state_interface name="effort"/>
       </joint>
       <joint name="arm_r_joint6">
@@ -102,4 +107,5 @@
         <state_interface name="position"/>
         <state_interface name="velocity"/>
+        <state_interface name="effort"/>
       </joint>
       <joint name="arm_r_joint7">
@@ -107,4 +113,5 @@
         <state_interface name="position"/>
         <state_interface name="velocity"/>
+        <state_interface name="effort"/>
       </joint>
       <joint name="gripper_r_joint1">
@@ -112,4 +119,5 @@
         <state_interface name="position"/>
         <state_interface name="velocity"/>
+        <state_interface name="effort"/>
       </joint>
       <joint name="arm_l_joint1">
@@ -117,4 +125,5 @@
         <state_interface name="position"/>
         <state_interface name="velocity"/>
+        <state_interface name="effort"/>
       </joint>
       <joint name="arm_l_joint2">
@@ -122,4 +131,5 @@
         <state_interface name="position"/>
         <state_interface name="velocity"/>
+        <state_interface name="effort"/>
       </joint>
       <joint name="arm_l_joint3">
@@ -127,4 +137,5 @@
         <state_interface name="position"/>
         <state_interface name="velocity"/>
+        <state_interface name="effort"/>
       </joint>
       <joint name="arm_l_joint4">
@@ -132,4 +143,5 @@
         <state_interface name="position"/>
         <state_interface name="velocity"/>
+        <state_interface name="effort"/>
       </joint>
       <joint name="arm_l_joint5">
@@ -137,4 +149,5 @@
         <state_interface name="position"/>
         <state_interface name="velocity"/>
+        <state_interface name="effort"/>
       </joint>
       <joint name="arm_l_joint6">
@@ -142,4 +155,5 @@
         <state_interface name="position"/>
         <state_interface name="velocity"/>
+        <state_interface name="effort"/>
       </joint>
       <joint name="arm_l_joint7">
@@ -147,4 +161,5 @@
         <state_interface name="position"/>
         <state_interface name="velocity"/>
+        <state_interface name="effort"/>
       </joint>
       <joint name="gripper_l_joint1">
@@ -152,4 +167,5 @@
         <state_interface name="position"/>
         <state_interface name="velocity"/>
+        <state_interface name="effort"/>
       </joint>
       <joint name="lift_joint">
@@ -157,4 +173,5 @@
         <state_interface name="position"/>
         <state_interface name="velocity"/>
+        <state_interface name="effort"/>
       </joint>
       <joint name="head_joint1">
@@ -162,4 +179,5 @@
         <state_interface name="position"/>
         <state_interface name="velocity"/>
+        <state_interface name="effort"/>
       </joint>
       <joint name="head_joint2">
@@ -167,4 +185,5 @@
         <state_interface name="position"/>
         <state_interface name="velocity"/>
+        <state_interface name="effort"/>
       </joint>
       <!-- RIGHT ARM -->
@@ -175,16 +194,20 @@
         <state_interface name="Present Position"/>
         <state_interface name="Present Velocity"/>
-        <param name="Drive Mode">1</param>
-        <param name="Operating Mode">3</param>
-        <param name="Return Delay Time">0</param>
-        <param name="Velocity Limit">2020</param>
-        <param name="Acceleration Limit">20200</param>
-        <param name="Profile Velocity">2020</param>
-        <param name="Profile Acceleration">300</param>
-        <param name="Max Position Limit">262144</param>
-        <param name="Min Position Limit">-262144</param>
-        <param name="Position P Gain">1583185</param>
-        <param name="Velocity P Gain">41387</param>
-        <param name="Velocity I Gain">1065630</param>
+        <state_interface name="Present Current"/>
+        <param name="Drive Mode">5</param>
+        <param name="Operating Mode">3</param>
+        <param name="Return Delay Time">0</param>
+        <param name="Velocity Limit">3591</param>
+        <param name="Acceleration Limit">35910</param>
+        <param name="Profile Velocity">3591</param>
+        <param name="Profile Acceleration">3591</param>
+        <param name="Profile Acceleration Time">250</param>
+        <param name="Profile Time">500</param>
+        <param name="Max Position Limit">262144</param>
+        <param name="Min Position Limit">-262144</param>
+        <param name="Position P Gain">1583185</param>
+        <param name="Velocity P Gain">41387</param>
+        <param name="Velocity I Gain">1565630</param>
+        <param name="Position FF Gain">100</param>
       </gpio>
       <gpio name="dxl2">
@@ -194,16 +217,20 @@
         <state_interface name="Present Position"/>
         <state_interface name="Present Velocity"/>
-        <param name="Drive Mode">0</param>
-        <param name="Operating Mode">3</param>
-        <param name="Return Delay Time">0</param>
-        <param name="Velocity Limit">2020</param>
-        <param name="Acceleration Limit">20200</param>
-        <param name="Profile Velocity">2020</param>
-        <param name="Profile Acceleration">300</param>
+        <state_interface name="Present Current"/>
+        <param name="Drive Mode">4</param>
+        <param name="Operating Mode">3</param>
+        <param name="Return Delay Time">0</param>
+        <param name="Velocity Limit">3591</param>
+        <param name="Acceleration Limit">35910</param>
+        <param name="Profile Velocity">3591</param>
+        <param name="Profile Acceleration">3591</param>
+        <param name="Profile Acceleration Time">250</param>
+        <param name="Profile Time">500</param>
         <param name="Max Position Limit">0</param>
         <param name="Min Position Limit">-262144</param>
         <param name="Position P Gain">1583185</param>
         <param name="Velocity P Gain">41387</param>
-        <param name="Velocity I Gain">1065630</param>
+        <param name="Velocity I Gain">1565630</param>
+        <param name="Position FF Gain">100</param>
       </gpio>
       <gpio name="dxl3">
@@ -213,16 +240,20 @@
         <state_interface name="Present Position"/>
         <state_interface name="Present Velocity"/>
-        <param name="Drive Mode">1</param>
-        <param name="Operating Mode">3</param>
-        <param name="Return Delay Time">0</param>
-        <param name="Velocity Limit">2020</param>
-        <param name="Acceleration Limit">20200</param>
-        <param name="Profile Velocity">2020</param>
-        <param name="Profile Acceleration">300</param>
-        <param name="Max Position Limit">262144</param>
-        <param name="Min Position Limit">-262144</param>
-        <param name="Position P Gain">1583185</param>
-        <param name="Velocity P Gain">41387</param>
-        <param name="Velocity I Gain">1065630</param>
+        <state_interface name="Present Current"/>
+        <param name="Drive Mode">5</param>
+        <param name="Operating Mode">3</param>
+        <param name="Return Delay Time">0</param>
+        <param name="Velocity Limit">3591</param>
+        <param name="Acceleration Limit">35910</param>
+        <param name="Profile Velocity">3591</param>
+        <param name="Profile Acceleration">3591</param>
+        <param name="Profile Acceleration Time">250</param>
+        <param name="Profile Time">500</param>
+        <param name="Max Position Limit">262144</param>
+        <param name="Min Position Limit">-262144</param>
+        <param name="Position P Gain">1583185</param>
+        <param name="Velocity P Gain">41387</param>
+        <param name="Velocity I Gain">1565630</param>
+        <param name="Position FF Gain">100</param>
       </gpio>
       <gpio name="dxl4">
@@ -232,16 +263,20 @@
         <state_interface name="Present Position"/>
         <state_interface name="Present Velocity"/>
-        <param name="Drive Mode">1</param>
-        <param name="Operating Mode">3</param>
-        <param name="Return Delay Time">0</param>
-        <param name="Velocity Limit">2020</param>
-        <param name="Acceleration Limit">20200</param>
-        <param name="Profile Velocity">2020</param>
-        <param name="Profile Acceleration">300</param>
+        <state_interface name="Present Current"/>
+        <param name="Drive Mode">5</param>
+        <param name="Operating Mode">3</param>
+        <param name="Return Delay Time">0</param>
+        <param name="Velocity Limit">6486</param>
+        <param name="Acceleration Limit">35910</param>
+        <param name="Profile Velocity">6486</param>
+        <param name="Profile Acceleration">3591</param>
+        <param name="Profile Acceleration Time">250</param>
+        <param name="Profile Time">500</param>
         <param name="Max Position Limit">90000</param>
         <param name="Min Position Limit">-245000</param>
         <param name="Position P Gain">1583185</param>
         <param name="Velocity P Gain">18184</param>
-        <param name="Velocity I Gain">1085331</param>
+        <param name="Velocity I Gain">1585331</param>
+        <param name="Position FF Gain">100</param>
       </gpio>
       <gpio name="dxl5">
@@ -251,16 +286,20 @@
         <state_interface name="Present Position"/>
         <state_interface name="Present Velocity"/>
-        <param name="Drive Mode">1</param>
-        <param name="Operating Mode">3</param>
-        <param name="Return Delay Time">0</param>
-        <param name="Velocity Limit">2020</param>
-        <param name="Acceleration Limit">20200</param>
-        <param name="Profile Velocity">2020</param>
-        <param name="Profile Acceleration">300</param>
+        <state_interface name="Present Current"/>
+        <param name="Drive Mode">5</param>
+        <param name="Operating Mode">3</param>
+        <param name="Return Delay Time">0</param>
+        <param name="Velocity Limit">6486</param>
+        <param name="Acceleration Limit">35910</param>
+        <param name="Profile Velocity">6486</param>
+        <param name="Profile Acceleration">3591</param>
+        <param name="Profile Acceleration Time">250</param>
+        <param name="Profile Time">500</param>
         <param name="Max Position Limit">262144</param>
         <param name="Min Position Limit">-262144</param>
         <param name="Position P Gain">1583185</param>
         <param name="Velocity P Gain">18184</param>
-        <param name="Velocity I Gain">1085331</param>
+        <param name="Velocity I Gain">1585331</param>
+        <param name="Position FF Gain">100</param>
       </gpio>
       <gpio name="dxl6">
@@ -270,16 +309,20 @@
         <state_interface name="Present Position"/>
         <state_interface name="Present Velocity"/>
-        <param name="Drive Mode">1</param>
-        <param name="Operating Mode">3</param>
-        <param name="Return Delay Time">0</param>
-        <param name="Velocity Limit">2020</param>
-        <param name="Acceleration Limit">20200</param>
-        <param name="Profile Velocity">2020</param>
-        <param name="Profile Acceleration">300</param>
+        <state_interface name="Present Current"/>
+        <param name="Drive Mode">5</param>
+        <param name="Operating Mode">3</param>
+        <param name="Return Delay Time">0</param>
+        <param name="Velocity Limit">6486</param>
+        <param name="Acceleration Limit">35910</param>
+        <param name="Profile Velocity">6486</param>
+        <param name="Profile Acceleration">3591</param>
+        <param name="Profile Acceleration Time">250</param>
+        <param name="Profile Time">500</param>
         <param name="Max Position Limit">131072</param>
         <param name="Min Position Limit">-131072</param>
         <param name="Position P Gain">1583185</param>
         <param name="Velocity P Gain">18184</param>
-        <param name="Velocity I Gain">1085331</param>
+        <param name="Velocity I Gain">1585331</param>
+        <param name="Position FF Gain">100</param>
       </gpio>
       <gpio name="dxl7">
@@ -289,12 +332,14 @@
         <state_interface name="Present Position"/>
         <state_interface name="Present Velocity"/>
-        <param name="Drive Mode">0</param>
-        <param name="Operating Mode">3</param>
-        <param name="Return Delay Time">0</param>
-        <param name="Velocity Limit">2020</param>
-        <param name="Profile Velocity">2020</param>
-        <param name="Profile Acceleration">3000</param>
-        <param name="Max Position Limit">151875</param>
-        <param name="Min Position Limit">-131875</param>
+        <state_interface name="Present Current"/>
+        <param name="Drive Mode">4</param>
+        <param name="Operating Mode">3</param>
+        <param name="Return Delay Time">0</param>
+        <param name="Velocity Limit">2920</param>
+        <param name="Acceleration Limit">359100</param>
+        <param name="Profile Velocity">100</param>
+        <param name="Profile Acceleration">50</param>
+        <param name="Max Position Limit">131875</param>
+        <param name="Min Position Limit">-151875</param>
       </gpio>
       <gpio name="dxl8">
@@ -304,4 +349,5 @@
         <state_interface name="Present Position"/>
         <state_interface name="Present Velocity"/>
+        <state_interface name="Present Current"/>
         <param name="Operating Mode">5</param>
         <param name="Return Delay Time">0</param>
@@ -316,16 +362,20 @@
         <state_interface name="Present Position"/>
         <state_interface name="Present Velocity"/>
-        <param name="Drive Mode">0</param>
-        <param name="Operating Mode">3</param>
-        <param name="Return Delay Time">0</param>
-        <param name="Velocity Limit">2020</param>
-        <param name="Acceleration Limit">20200</param>
-        <param name="Profile Velocity">2020</param>
-        <param name="Profile Acceleration">300</param>
-        <param name="Max Position Limit">262144</param>
-        <param name="Min Position Limit">-262144</param>
-        <param name="Position P Gain">1583185</param>
-        <param name="Velocity P Gain">41387</param>
-        <param name="Velocity I Gain">1065630</param>
+        <state_interface name="Present Current"/>
+        <param name="Drive Mode">4</param>
+        <param name="Operating Mode">3</param>
+        <param name="Return Delay Time">0</param>
+        <param name="Velocity Limit">3591</param>
+        <param name="Acceleration Limit">35910</param>
+        <param name="Profile Velocity">3591</param>
+        <param name="Profile Acceleration">3591</param>
+        <param name="Profile Acceleration Time">250</param>
+        <param name="Profile Time">500</param>
+        <param name="Max Position Limit">262144</param>
+        <param name="Min Position Limit">-262144</param>
+        <param name="Position P Gain">1583185</param>
+        <param name="Velocity P Gain">41387</param>
+        <param name="Velocity I Gain">1565630</param>
+        <param name="Position FF Gain">100</param>
       </gpio>
       <gpio name="dxl32">
@@ -335,16 +385,20 @@
         <state_interface name="Present Position"/>
         <state_interface name="Present Velocity"/>
-        <param name="Drive Mode">0</param>
-        <param name="Operating Mode">3</param>
-        <param name="Return Delay Time">0</param>
-        <param name="Velocity Limit">2020</param>
-        <param name="Acceleration Limit">20200</param>
-        <param name="Profile Velocity">2020</param>
-        <param name="Profile Acceleration">300</param>
+        <state_interface name="Present Current"/>
+        <param name="Drive Mode">4</param>
+        <param name="Operating Mode">3</param>
+        <param name="Return Delay Time">0</param>
+        <param name="Velocity Limit">3591</param>
+        <param name="Acceleration Limit">35910</param>
+        <param name="Profile Velocity">3591</param>
+        <param name="Profile Acceleration">3591</param>
+        <param name="Profile Acceleration Time">250</param>
+        <param name="Profile Time">500</param>
         <param name="Max Position Limit">262144</param>
         <param name="Min Position Limit">0</param>
         <param name="Position P Gain">1583185</param>
         <param name="Velocity P Gain">41387</param>
-        <param name="Velocity I Gain">1065630</param>
+        <param name="Velocity I Gain">1565630</param>
+        <param name="Position FF Gain">100</param>
       </gpio>
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
File: ffw_description/ros2_control/ffw_lg2_leader/ffw_lg2_leader_left.ros2_control.xacro (robot description, xacro)
@@ -23,4 +23,5 @@
             <param name="number_of_joints">8</param>
             <param name="number_of_transmissions">8</param>
+            <param name="disable_torque_at_init">true</param>
             <param name="transmission_to_joint_matrix">
               1, 0, 0, 0, 0, 0, 0, 0,

File: ffw_description/ros2_control/ffw_lg2_leader/ffw_lg2_leader_right.ros2_control.xacro (robot description, xacro)
@@ -23,4 +23,5 @@
             <param name="number_of_joints">8</param>
             <param name="number_of_transmissions">8</param>
+            <param name="disable_torque_at_init">true</param>
             <param name="transmission_to_joint_matrix">
               1, 0, 0, 0, 0, 0, 0, 0,
