Commit message: Imported upstream version '1.0.9' of 'upstream'

File: ffw_description/urdf/common/follower/ffw_follower_body.xacro (robot description, xacro)
@@ -28,4 +28,11 @@
             </geometry>
          </collision>
+         <inertial>
+            <origin xyz="-1.492287800e-02 2.731522500e-03 -4.342526400e-02" />
+            <mass value="6.193955900e+00" />
+            <inertia ixx="1.082886600e-01" ixy="2.929692500e-06" ixz="-1.572750800e-03"
+            iyy="5.432369700e-02" iyz="1.698970600e-03"
+            izz="7.960084300e-02" />
+         </inertial>
       </link>
       <joint name="${prefix}head_joint1" type="revolute">
@@ -53,4 +60,11 @@
             </geometry>
          </collision>
+         <inertial>
+            <origin xyz="2.533965600e-02 0.000000000e+00 4.774514600e-02" />
+            <mass value="1.235180200e-01" />
+            <inertia ixx="6.870965700e-03" ixy="8.592260200e-07" ixz="-3.002664500e-04"
+            iyy="1.771510200e-02" iyz="-4.447973700e-07"
+            izz="1.631113500e-02" />
+         </inertial>
       </link>
       <joint name="${prefix}head_joint2" type="revolute">
@@ -78,4 +92,11 @@
             </geometry>
          </collision>
+         <inertial>
+            <origin xyz="3.052563400e-03 1.180475700e-03 -1.593280400e-02" />
+            <mass value="3.254213000e-01" />
+            <inertia ixx="8.907301100e-04" ixy="-5.211330800e-06" ixz="1.758054200e-05"
+            iyy="7.631788100e-04" iyz="-1.022156300e-06"
+            izz="1.339403400e-03" />
+         </inertial>
       </link>
       <joint name="${prefix}arm_l_joint1" type="revolute">
@@ -103,4 +124,11 @@
             </geometry>
          </collision>
+         <inertial>
+            <origin xyz="1.421037300e-02 1.155371800e-01 1.120644000e-04" />
+            <mass value="2.001332200e+00" />
+            <inertia ixx="2.507557700e-03" ixy="-2.196355800e-04" ixz="1.151251900e-05"
+            iyy="2.865299700e-03" iyz="-2.311007900e-06"
+            izz="3.365371600e-03" />
+         </inertial>
       </link>
       <joint name="${prefix}arm_l_joint2" type="revolute">
@@ -128,4 +156,11 @@
             </geometry>
          </collision>
+         <inertial>
+            <origin xyz="9.109841300e-03 -1.053016500e-04 -1.438640700e-01" />
+            <mass value="2.128261000e+00" />
+            <inertia ixx="9.976166600e-03" ixy="-1.420641600e-06" ixz="-2.370609000e-03"
+            iyy="1.088835300e-02" iyz="4.832141500e-06"
+            izz="3.168582700e-03" />
+         </inertial>
       </link>
       <joint name="${prefix}arm_l_joint3" type="revolute">
@@ -153,4 +188,11 @@
             </geometry>
          </collision>
+         <inertial>
+            <origin xyz="2.987537300e-02 1.391394900e-02 -1.210139000e-01" />
+            <mass value="1.684755100e+00" />
+            <inertia ixx="2.878077200e-03" ixy="-2.615265200e-04" ixz="6.679408300e-04"
+            iyy="2.707096100e-03" iyz="3.296252200e-04"
+            izz="2.566350600e-03" />
+         </inertial>
       </link>
       <joint name="${prefix}arm_l_joint4" type="revolute">
@@ -178,4 +220,11 @@
             </geometry>
          </collision>
+         <inertial>
+            <origin xyz="-3.853865300e-02 9.807228600e-03 -1.313122800e-01" />
+            <mass value="1.508214400e+00" />
+            <inertia ixx="6.252303800e-03" ixy="-2.162798200e-04" ixz="-5.113660100e-04"
+            iyy="5.705086400e-03" iyz="-1.597759100e-03"
+            izz="2.098027800e-03" />
+         </inertial>
       </link>
       <joint name="${prefix}arm_l_joint5" type="revolute">
@@ -203,4 +252,11 @@
             </geometry>
          </collision>
+         <inertial>
+            <origin xyz="-3.122616100e-05 1.681922700e-02 -9.873815600e-02" />
+            <mass value="1.391783100e+00" />
+            <inertia ixx="1.885672100e-03" ixy="1.326915800e-06" ixz="2.418484800e-07"
+            iyy="1.285272900e-03" iyz="1.287761700e-04"
+            izz="1.689335300e-03" />
+         </inertial>
       </link>
       <joint name="${prefix}arm_l_joint6" type="revolute">
@@ -228,4 +284,11 @@
             </geometry>
          </collision>
+         <inertial>
+            <origin xyz="2.243891700e-03 1.876410500e-02 -6.480557600e-02" />
+            <mass value="6.577074100e-01" />
+            <inertia ixx="1.416138700e-03" ixy="2.839010300e-05" ixz="3.582229500e-05"
+            iyy="1.142334400e-03" iyz="-5.356836800e-04"
+            izz="1.017517600e-03" />
+         </inertial>
       </link>
       <joint name="${prefix}arm_l_joint7" type="revolute">
@@ -253,4 +316,11 @@
             </geometry>
          </collision>
+         <inertial>
+            <origin xyz="2.550659300e-02 0.000000000e+00 -5.539533100e-02" />
+            <mass value="1.668563000e-01" />
+            <inertia ixx="1.035867900e-04" ixy="0.000000000e+00" ixz="1.098870100e-05"
+            iyy="4.524528700e-04" iyz="0.000000000e+00"
+            izz="4.156884400e-04" />
+         </inertial>
       </link>
       <xacro:sensor_d405 parent="${prefix}arm_l_link7" use_nominal_extrinsics="false" name="${prefix}camera_l">
@@ -281,4 +351,11 @@
             </geometry>
          </collision>
+         <inertial>
+            <origin xyz="1.421037300e-02 -1.155371800e-01 -1.120644000e-04" />
+            <mass value="2.001332200e+00" />
+            <inertia ixx="2.507557700e-03" ixy="2.196355800e-04" ixz="-1.151251900e-05"
+            iyy="2.865299700e-03" iyz="-2.311007900e-06"
+            izz="3.365371600e-03" />
+         </inertial>
       </link>
       <joint name="${prefix}arm_r_joint2" type="revolute">
@@ -306,4 +383,11 @@
             </geometry>
          </collision>
+         <inertial>
+            <origin xyz="9.109841300e-03 -1.053016500e-04 -1.438640700e-01" />
+            <mass value="2.128261000e+00" />
+            <inertia ixx="9.976166600e-03" ixy="-1.420641600e-06" ixz="-2.370609000e-03"
+            iyy="1.088835300e-02" iyz="4.832141500e-06"
+            izz="3.168582700e-03" />
+         </inertial>
       </link>
       <joint name="${prefix}arm_r_joint3" type="revolute">
@@ -331,4 +415,11 @@
             </geometry>
          </collision>
+         <inertial>
+            <origin xyz="2.984576500e-02 -1.392295900e-02 -1.210435100e-01" />
+            <mass value="1.684755100e+00" />
+            <inertia ixx="2.877971200e-03" ixy="2.632159900e-04" ixz="6.677998500e-04"
+            iyy="2.707378400e-03" iyz="-3.275929900e-04"
+            izz="2.563528600e-03" />
+         </inertial>
       </link>
       <joint name="${prefix}arm_r_joint4" type="revolute">
@@ -356,4 +447,11 @@
             </geometry>
          </collision>
+         <inertial>
+            <origin xyz="-3.867746800e-02 -9.308009900e-03 -1.322971300e-01" />
+            <mass value="1.494251100e+00" />
+            <inertia ixx="6.032357900e-03" ixy="2.028997300e-04" ixz="-4.854051900e-04"
+            iyy="5.536423500e-03" iyz="1.507124600e-03"
+            izz="2.032999700e-03" />
+         </inertial>
       </link>
       <joint name="${prefix}arm_r_joint5" type="revolute">
@@ -381,4 +479,11 @@
             </geometry>
          </collision>
+         <inertial>
+            <origin xyz="8.387686000e-04 -1.679849900e-02 -9.873815600e-02" />
+            <mass value="1.391783100e+00" />
+            <inertia ixx="1.882492800e-03" ixy="3.480391000e-05" ixz="6.806743100e-06"
+            iyy="1.288452200e-03" iyz="-1.285963700e-04"
+            izz="1.689335300e-03" />
+         </inertial>
       </link>
       <joint name="${prefix}arm_r_joint6" type="revolute">
@@ -406,4 +511,11 @@
             </geometry>
          </collision>
+         <inertial>
+            <origin xyz="3.267491200e-03 -1.861259000e-02 -6.479261600e-02" />
+            <mass value="6.577074100e-01" />
+            <inertia ixx="1.417976200e-03" ixy="-1.325841000e-05" ixz="6.534407900e-06"
+            iyy="1.139647400e-03" iyz="5.366707300e-04"
+            izz="1.017476200e-03" />
+         </inertial>
       </link>
       <joint name="${prefix}arm_r_joint7" type="revolute">
@@ -431,4 +543,11 @@
             </geometry>
          </collision>
+         <inertial>
+            <origin xyz="2.546836200e-02 1.396001200e-03 -5.539533100e-02" />
+            <mass value="1.668563000e-01" />
+            <inertia ixx="1.046318100e-04" ixy="-1.906515900e-05" ixz="1.097223300e-05"
+            iyy="4.514078500e-04" iyz="6.013716400e-07"
+            izz="4.156884400e-04" />
+         </inertial>
       </link>
       <xacro:sensor_d405 parent="${prefix}arm_r_link7" use_nominal_extrinsics="false" name="${prefix}camera_r">

File: ffw_description/urdf/ffw_bg2_rev4_follower/ffw_bg2_follower.urdf (robot description, URDF)
Before this commit: robot ffw_bg2_follower, 33 links, 32 joints
Links:
- link arm_base_link: mass None -> 6.193955900e+00
- link arm_l_link1: mass None -> 2.001332200e+00
- link arm_l_link2: mass None -> 2.128261000e+00
- link arm_l_link3: mass None -> 1.684755100e+00
- link arm_l_link4: mass None -> 1.508214400e+00
- link arm_l_link5: mass None -> 1.391783100e+00
- link arm_l_link6: mass None -> 6.577074100e-01
- link arm_l_link7: mass None -> 1.668563000e-01
- link arm_r_link1: mass None -> 2.001332200e+00
- link arm_r_link2: mass None -> 2.128261000e+00
- link arm_r_link3: mass None -> 1.684755100e+00
- link arm_r_link4: mass None -> 1.494251100e+00
- link arm_r_link5: mass None -> 1.391783100e+00
- link arm_r_link6: mass None -> 6.577074100e-01
- link arm_r_link7: mass None -> 1.668563000e-01
- link base_link: mass None -> 5.435831600e+01
- link head_link1: mass None -> 1.235180200e-01
- link head_link2: mass None -> 3.254213000e-01

File: ffw_description/urdf/ffw_bg2_rev4_follower/ffw_bg2_follower.urdf.xacro (robot description, xacro)
@@ -19,18 +19,25 @@
   <link name="$(arg prefix)base_link">
     <visual>
-        <origin xyz="0 0 0" rpy="0 0 0" />
-        <geometry>
-          <mesh filename="${meshes_file_direction}/base_mobile_assy.stl" scale="0.001 0.001 0.001" />
-        </geometry>
-          <material name="silver">
-              <color rgba="0.75 0.75 0.75 1"/>
-          </material>
+      <origin xyz="0 0 0" rpy="0 0 0" />
+      <geometry>
+        <mesh filename="${meshes_file_direction}/base_mobile_assy.stl" scale="0.001 0.001 0.001" />
+      </geometry>
+      <material name="silver">
+        <color rgba="0.75 0.75 0.75 1"/>
+      </material>
     </visual>
     <collision>
-        <origin xyz="0 0 0" rpy="0 0 0" />
-        <geometry>
-          <mesh filename="${meshes_file_direction}/base_mobile_assy.stl" scale="0.001 0.001 0.001" />
-        </geometry>
+      <origin xyz="0 0 0" rpy="0 0 0" />
+      <geometry>
+        <mesh filename="${meshes_file_direction}/base_mobile_assy.stl" scale="0.001 0.001 0.001" />
+      </geometry>
     </collision>
+    <inertial>
+      <origin xyz="-8.880608700e-03 -4.758427800e-03 3.886366400e-01" />
+      <mass value="5.435831600e+01" />
+      <inertia ixx="1.188633900e+06" ixy="6.334393100e+02" ixz="-1.454811600e+05"
+      iyy="1.090949100e+06" iyz="-5.126785200e+03"
+      izz="4.492808000e+05" />
+    </inertial>
   </link>
   <xacro:ffw_follower_body parent="$(arg prefix)base_link" prefix="$(arg prefix)">

Commit message: Imported upstream version '1.1.10' of 'upstream'

File: ffw_description/urdf/common/follower/ffw_follower_body.xacro (robot description, xacro)
@@ -3,4 +3,5 @@
    <xacro:macro name="ffw_follower_body" params="prefix parent *origin">
       <xacro:include filename="$(find realsense2_description)/urdf/_d405.urdf.xacro" />
+      <xacro:include filename="$(find ffw_description)/urdf/common/follower/zedm.urdf.xacro" />
       <xacro:property name="meshes_file_direction" value="package://ffw_description/meshes/common/follower" />
       <joint name="${prefix}lift_joint" type="prismatic">
@@ -39,5 +40,5 @@
          <parent link="${prefix}arm_base_link" />
          <child link="${prefix}head_link1" />
-         <origin xyz="0.0494878 0 0.102123" rpy="0 0 0" />
+         <origin xyz="0.049483 0 0.102130" rpy="0 0 0" />
          <axis xyz="0 1 0" />
          <limit velocity="4.8" effort="1000" lower="-0.2317" upper="0.6951" />
@@ -71,5 +72,5 @@
          <parent link="${prefix}head_link1" />
          <child link="${prefix}head_link2" />
-         <origin xyz="0.0365694 0 0.0563797" rpy="0 0 0" />
+         <origin xyz="0.040 0 0.054" rpy="0 0 0" />
          <axis xyz="0 0 1" />
          <limit velocity="4.8" effort="1000" lower="-0.35" upper="0.35" />
@@ -100,4 +101,10 @@
          </inertial>
       </link>
+      <xacro:zed_camera name="zedm" model="zedm" />
+      <joint name="zedm_joint" type="fixed">
+         <parent link="head_link2"/>
+         <child link="zedm_camera_link"/>
+         <origin xyz="0.0238122 -0.00651797 -0.0242094" rpy="0 0 0" />
+      </joint>
       <joint name="${prefix}arm_l_joint1" type="revolute">
          <parent link="${prefix}arm_base_link" />

File: ffw_description/urdf/ffw_bg2_rev2_follower/ffw_bg2_follower.urdf.xacro (robot description, xacro)
@@ -43,8 +43,8 @@
   </xacro:ffw_follower_body>
   <xacro:rh_p12_rn_a parent="$(arg prefix)arm_l_link7" prefix="$(arg prefix)gripper_l_">
-    <origin xyz="0 0 -0.05" rpy="0 3.14159265359 0"/>
+    <origin xyz="0 0 -0.05" rpy="0 3.14159265359 3.14159265359"/>
   </xacro:rh_p12_rn_a>
   <xacro:rh_p12_rn_a parent="$(arg prefix)arm_r_link7" prefix="$(arg prefix)gripper_r_">
-    <origin xyz="0 0 -0.05" rpy="0 3.14159265359 0"/>
+    <origin xyz="0 0 -0.05" rpy="0 3.14159265359 3.14159265359"/>
   </xacro:rh_p12_rn_a>
   <xacro:ffw_bg2_follower_system

File: ffw_description/urdf/ffw_bg2_rev3_follower/ffw_bg2_follower.urdf.xacro (robot description, xacro)
@@ -43,8 +43,8 @@
   </xacro:ffw_follower_body>
   <xacro:rh_p12_rn_a parent="$(arg prefix)arm_l_link7" prefix="$(arg prefix)gripper_l_">
-    <origin xyz="0 0 -0.05" rpy="0 3.14159265359 0"/>
+    <origin xyz="0 0 -0.05" rpy="0 3.14159265359 3.14159265359"/>
   </xacro:rh_p12_rn_a>
   <xacro:rh_p12_rn_a parent="$(arg prefix)arm_r_link7" prefix="$(arg prefix)gripper_r_">
-    <origin xyz="0 0 -0.05" rpy="0 3.14159265359 0"/>
+    <origin xyz="0 0 -0.05" rpy="0 3.14159265359 3.14159265359"/>
   </xacro:rh_p12_rn_a>
   <xacro:ffw_bg2_follower_system

File: ffw_description/urdf/ffw_bg2_rev4_follower/ffw_bg2_follower.urdf.xacro (robot description, xacro)
@@ -45,9 +45,41 @@
   </xacro:ffw_follower_body>
   <xacro:rh_p12_rn_a parent="$(arg prefix)arm_l_link7" prefix="$(arg prefix)gripper_l_">
-    <origin xyz="0 0 -0.078" rpy="0 3.14159265359 0"/>
+    <origin xyz="0 0 -0.078" rpy="0 3.14159265359 3.14159265359"/>
   </xacro:rh_p12_rn_a>
+  <joint name="$(arg prefix)end_effector_l_joint" type="fixed">
+    <parent link="$(arg prefix)arm_l_link7"/>
+    <child link="$(arg prefix)end_effector_l_link"/>
+    <origin xyz="0 0 -0.215" rpy="0 0 0"/>
+  </joint>
+  <link name="$(arg prefix)end_effector_l_link">
+    <visual>
+      <origin xyz="0 0 0" rpy="0 0 0"/>
+      <geometry>
+        <box size="0.01 0.01 0.01" />
+      </geometry>
+      <material name="red">
+        <color rgba="1.0 0.0 0.0 1"/>
+      </material>
+    </visual>
+  </link>
   <xacro:rh_p12_rn_a parent="$(arg prefix)arm_r_link7" prefix="$(arg prefix)gripper_r_">
-    <origin xyz="0 0 -0.078" rpy="0 3.14159265359 0"/>
+    <origin xyz="0 0 -0.078" rpy="0 3.14159265359 3.14159265359"/>
   </xacro:rh_p12_rn_a>
+  <joint name="$(arg prefix)end_effector_r_joint" type="fixed">
+    <parent link="$(arg prefix)arm_r_link7"/>
+    <child link="$(arg prefix)end_effector_r_link"/>
+    <origin xyz="0 0 -0.215" rpy="0 0 0"/>
+  </joint>
+  <link name="$(arg prefix)end_effector_r_link">
+    <visual>
+      <origin xyz="0 0 0" rpy="0 0 0"/>
+      <geometry>
+        <box size="0.01 0.01 0.01" />
+      </geometry>
+      <material name="red">
+        <color rgba="1.0 0.0 0.0 1"/>
+      </material>
+    </visual>
+  </link>
   <xacro:ffw_bg2_follower_system
     use_sim="$(arg use_sim)"

File: ffw_description/urdf/ffw_sg2_rev1_follower/ffw_sg2_follower.urdf.xacro (robot description, xacro)
@@ -72,7 +72,39 @@
     <origin xyz="0 0 -0.078" rpy="0 3.14159265359 3.14159265359"/>
   </xacro:rh_p12_rn_a>
+  <joint name="$(arg prefix)end_effector_l_joint" type="fixed">
+    <parent link="$(arg prefix)arm_l_link7"/>
+    <child link="$(arg prefix)end_effector_l_link"/>
+    <origin xyz="0 0 -0.215" rpy="0 0 0"/>
+  </joint>
+  <link name="$(arg prefix)end_effector_l_link">
+    <visual>
+      <origin xyz="0 0 0" rpy="0 0 0"/>
+      <geometry>
+        <box size="0.01 0.01 0.01" />
+      </geometry>
+      <material name="red">
+        <color rgba="1.0 0.0 0.0 1"/>
+      </material>
+    </visual>
+  </link>
   <xacro:rh_p12_rn_a parent="$(arg prefix)arm_r_link7" prefix="$(arg prefix)gripper_r_">
     <origin xyz="0 0 -0.078" rpy="0 3.14159265359 3.14159265359"/>
   </xacro:rh_p12_rn_a>
+  <joint name="$(arg prefix)end_effector_r_joint" type="fixed">
+    <parent link="$(arg prefix)arm_r_link7"/>
+    <child link="$(arg prefix)end_effector_r_link"/>
+    <origin xyz="0 0 -0.215" rpy="0 0 0"/>
+  </joint>
+  <link name="$(arg prefix)end_effector_r_link">
+    <visual>
+      <origin xyz="0 0 0" rpy="0 0 0"/>
+      <geometry>
+        <box size="0.01 0.01 0.01" />
+      </geometry>
+      <material name="red">
+        <color rgba="1.0 0.0 0.0 1"/>
+      </material>
+    </visual>
+  </link>
   <joint name="$(arg prefix)left_wheel_steer" type="revolute">
       <parent link="$(arg prefix)base_link"/>
