Commit message: Rebase from 'release/jazzy/ffw_description'

File: ros2_control/ffw_bg2_rev4_follower/ffw_bg2_follower.ros2_control.xacro (robot description, xacro)
@@ -196,5 +196,5 @@
         <state_interface name="Present Current"/>
         <state_interface name="Error Code"/>
-        <param name="Drive Mode">5</param>
+        <param name="Drive Mode">69</param>
         <param name="Operating Mode">3</param>
         <param name="Return Delay Time">0</param>
@@ -220,5 +220,5 @@
         <state_interface name="Present Current"/>
         <state_interface name="Error Code"/>
-        <param name="Drive Mode">4</param>
+        <param name="Drive Mode">68</param>
         <param name="Operating Mode">3</param>
         <param name="Return Delay Time">0</param>
@@ -244,5 +244,5 @@
         <state_interface name="Present Current"/>
         <state_interface name="Error Code"/>
-        <param name="Drive Mode">5</param>
+        <param name="Drive Mode">69</param>
         <param name="Operating Mode">3</param>
         <param name="Return Delay Time">0</param>
@@ -268,5 +268,5 @@
         <state_interface name="Present Current"/>
         <state_interface name="Error Code"/>
-        <param name="Drive Mode">5</param>
+        <param name="Drive Mode">69</param>
         <param name="Operating Mode">3</param>
         <param name="Return Delay Time">0</param>
@@ -292,5 +292,5 @@
         <state_interface name="Present Current"/>
         <state_interface name="Error Code"/>
-        <param name="Drive Mode">5</param>
+        <param name="Drive Mode">69</param>
         <param name="Operating Mode">3</param>
         <param name="Return Delay Time">0</param>
@@ -316,5 +316,5 @@
         <state_interface name="Present Current"/>
         <state_interface name="Error Code"/>
-        <param name="Drive Mode">5</param>
+        <param name="Drive Mode">69</param>
         <param name="Operating Mode">3</param>
         <param name="Return Delay Time">0</param>
@@ -373,5 +373,5 @@
         <state_interface name="Present Current"/>
         <state_interface name="Error Code"/>
-        <param name="Drive Mode">4</param>
+        <param name="Drive Mode">68</param>
         <param name="Operating Mode">3</param>
         <param name="Return Delay Time">0</param>
@@ -397,5 +397,5 @@
         <state_interface name="Present Current"/>
         <state_interface name="Error Code"/>
-        <param name="Drive Mode">4</param>
+        <param name="Drive Mode">68</param>
         <param name="Operating Mode">3</param>
         <param name="Return Delay Time">0</param>
@@ -421,5 +421,5 @@
         <state_interface name="Present Current"/>
         <state_interface name="Error Code"/>
-        <param name="Drive Mode">5</param>
+        <param name="Drive Mode">69</param>
         <param name="Operating Mode">3</param>
         <param name="Return Delay Time">0</param>
@@ -445,5 +445,5 @@
         <state_interface name="Present Current"/>
         <state_interface name="Error Code"/>
-        <param name="Drive Mode">4</param>
+        <param name="Drive Mode">68</param>
         <param name="Operating Mode">3</param>
         <param name="Return Delay Time">0</param>
@@ -469,5 +469,5 @@
         <state_interface name="Present Current"/>
         <state_interface name="Error Code"/>
-        <param name="Drive Mode">5</param>
+        <param name="Drive Mode">69</param>
         <param name="Operating Mode">3</param>
         <param name="Return Delay Time">0</param>
@@ -493,5 +493,5 @@
         <state_interface name="Present Current"/>
         <state_interface name="Error Code"/>
-        <param name="Drive Mode">4</param>
+        <param name="Drive Mode">68</param>
         <param name="Operating Mode">3</param>
         <param name="Return Delay Time">0</param>

File: ros2_control/ffw_sg2_rev1_follower/ffw_sg2_follower.ros2_control.xacro (robot description, xacro)
@@ -220,5 +220,5 @@
         <state_interface name="Present Current"/>
         <state_interface name="Error Code"/>
-        <param name="Drive Mode">5</param>
+        <param name="Drive Mode">69</param>
         <param name="Operating Mode">3</param>
         <param name="Return Delay Time">0</param>
@@ -244,5 +244,5 @@
         <state_interface name="Present Current"/>
         <state_interface name="Error Code"/>
-        <param name="Drive Mode">4</param>
+        <param name="Drive Mode">68</param>
         <param name="Operating Mode">3</param>
         <param name="Return Delay Time">0</param>
@@ -268,5 +268,5 @@
         <state_interface name="Present Current"/>
         <state_interface name="Error Code"/>
-        <param name="Drive Mode">5</param>
+        <param name="Drive Mode">69</param>
         <param name="Operating Mode">3</param>
         <param name="Return Delay Time">0</param>
@@ -292,5 +292,5 @@
         <state_interface name="Present Current"/>
         <state_interface name="Error Code"/>
-        <param name="Drive Mode">5</param>
+        <param name="Drive Mode">69</param>
         <param name="Operating Mode">3</param>
         <param name="Return Delay Time">0</param>
@@ -316,5 +316,5 @@
         <state_interface name="Present Current"/>
         <state_interface name="Error Code"/>
-        <param name="Drive Mode">5</param>
+        <param name="Drive Mode">69</param>
         <param name="Operating Mode">3</param>
         <param name="Return Delay Time">0</param>
@@ -340,5 +340,5 @@
         <state_interface name="Present Current"/>
         <state_interface name="Error Code"/>
-        <param name="Drive Mode">5</param>
+        <param name="Drive Mode">69</param>
         <param name="Operating Mode">3</param>
         <param name="Return Delay Time">0</param>
@@ -397,5 +397,5 @@
         <state_interface name="Present Current"/>
         <state_interface name="Error Code"/>
-        <param name="Drive Mode">4</param>
+        <param name="Drive Mode">68</param>
         <param name="Operating Mode">3</param>
         <param name="Return Delay Time">0</param>
@@ -421,5 +421,5 @@
         <state_interface name="Present Current"/>
         <state_interface name="Error Code"/>
-        <param name="Drive Mode">4</param>
+        <param name="Drive Mode">68</param>
         <param name="Operating Mode">3</param>
         <param name="Return Delay Time">0</param>
@@ -445,5 +445,5 @@
         <state_interface name="Present Current"/>
         <state_interface name="Error Code"/>
-        <param name="Drive Mode">5</param>
+        <param name="Drive Mode">69</param>
         <param name="Operating Mode">3</param>
         <param name="Return Delay Time">0</param>
@@ -469,5 +469,5 @@
         <state_interface name="Present Current"/>
         <state_interface name="Error Code"/>
-        <param name="Drive Mode">4</param>
+        <param name="Drive Mode">68</param>
         <param name="Operating Mode">3</param>
         <param name="Return Delay Time">0</param>
@@ -493,5 +493,5 @@
         <state_interface name="Present Current"/>
         <state_interface name="Error Code"/>
-        <param name="Drive Mode">5</param>
+        <param name="Drive Mode">69</param>
         <param name="Operating Mode">3</param>
         <param name="Return Delay Time">0</param>
@@ -517,5 +517,5 @@
         <state_interface name="Present Current"/>
         <state_interface name="Error Code"/>
-        <param name="Drive Mode">4</param>
+        <param name="Drive Mode">68</param>
         <param name="Operating Mode">3</param>
         <param name="Return Delay Time">0</param>

File: urdf/common/follower/zedm.urdf.xacro (robot description, xacro)
@@ -29,5 +29,5 @@
 			<parent link="${name}_camera_center"/>
 			<child link="${name}_left_camera_frame"/>
-			<origin xyz="0 0.063 0" rpy="0 0 0" />
+			<origin xyz="0 0.0315 0" rpy="0 0 0" />
 		</joint>
 		<link name="${name}_left_camera_optical_frame"/>
@@ -41,5 +41,5 @@
 			<parent link="${name}_camera_center"/>
 			<child link="${name}_right_camera_frame"/>
-			<origin xyz="0 -0.063 0" rpy="0 0 0" />
+			<origin xyz="0 -0.0315 0" rpy="0 0 0" />
 		</joint>
 		<link name="${name}_right_camera_optical_frame"/>
