Commit message: Rebase from 'upstream'

File: ffw_description/ros2_control/ffw_bg2_rev2_follower/ffw_bg2_follower.ros2_control.xacro (robot description, xacro)
@@ -195,4 +195,5 @@
         <state_interface name="Present Velocity"/>
         <state_interface name="Present Current"/>
+        <state_interface name="Error Code"/>
         <param name="Drive Mode">5</param>
         <param name="Operating Mode">3</param>
@@ -218,4 +219,5 @@
         <state_interface name="Present Velocity"/>
         <state_interface name="Present Current"/>
+        <state_interface name="Error Code"/>
         <param name="Drive Mode">4</param>
         <param name="Operating Mode">3</param>
@@ -241,4 +243,5 @@
         <state_interface name="Present Velocity"/>
         <state_interface name="Present Current"/>
+        <state_interface name="Error Code"/>
         <param name="Drive Mode">5</param>
         <param name="Operating Mode">3</param>
@@ -264,4 +267,5 @@
         <state_interface name="Present Velocity"/>
         <state_interface name="Present Current"/>
+        <state_interface name="Error Code"/>
         <param name="Drive Mode">5</param>
         <param name="Operating Mode">3</param>
@@ -287,4 +291,5 @@
         <state_interface name="Present Velocity"/>
         <state_interface name="Present Current"/>
+        <state_interface name="Error Code"/>
         <param name="Drive Mode">5</param>
         <param name="Operating Mode">3</param>
@@ -310,4 +315,5 @@
         <state_interface name="Present Velocity"/>
         <state_interface name="Present Current"/>
+        <state_interface name="Error Code"/>
         <param name="Drive Mode">5</param>
         <param name="Operating Mode">3</param>
@@ -333,4 +339,5 @@
         <state_interface name="Present Velocity"/>
         <state_interface name="Present Current"/>
+        <state_interface name="Hardware Error Status"/>
         <param name="Drive Mode">5</param>
         <param name="Operating Mode">3</param>
@@ -351,4 +358,5 @@
         <state_interface name="Present Velocity"/>
         <state_interface name="Present Current"/>
+        <state_interface name="Hardware Error Status"/>
         <param name="Operating Mode">5</param>
         <param name="Return Delay Time">0</param>
@@ -364,4 +372,5 @@
         <state_interface name="Present Velocity"/>
         <state_interface name="Present Current"/>
+        <state_interface name="Error Code"/>
         <param name="Drive Mode">4</param>
         <param name="Operating Mode">3</param>
@@ -387,4 +396,5 @@
         <state_interface name="Present Velocity"/>
         <state_interface name="Present Current"/>
+        <state_interface name="Error Code"/>
         <param name="Drive Mode">4</param>
         <param name="Operating Mode">3</param>
@@ -410,4 +420,5 @@
         <state_interface name="Present Velocity"/>
         <state_interface name="Present Current"/>
+        <state_interface name="Error Code"/>
         <param name="Drive Mode">5</param>
         <param name="Operating Mode">3</param>
@@ -433,4 +444,5 @@
         <state_interface name="Present Velocity"/>
         <state_interface name="Present Current"/>
+        <state_interface name="Error Code"/>
         <param name="Drive Mode">4</param>
         <param name="Operating Mode">3</param>
@@ -456,4 +468,5 @@
         <state_interface name="Present Velocity"/>
         <state_interface name="Present Current"/>
+        <state_interface name="Error Code"/>
         <param name="Drive Mode">5</param>
         <param name="Operating Mode">3</param>
@@ -479,4 +492,5 @@
         <state_interface name="Present Velocity"/>
         <state_interface name="Present Current"/>
+        <state_interface name="Error Code"/>
         <param name="Drive Mode">4</param>
         <param name="Operating Mode">3</param>
@@ -502,4 +516,5 @@
         <state_interface name="Present Velocity"/>
         <state_interface name="Present Current"/>
+        <state_interface name="Hardware Error Status"/>
         <param name="Drive Mode">5</param>
         <param name="Operating Mode">3</param>
@@ -520,4 +535,5 @@
         <state_interface name="Present Velocity"/>
         <state_interface name="Present Current"/>
+        <state_interface name="Hardware Error Status"/>
         <param name="Operating Mode">5</param>
         <param name="Return Delay Time">0</param>
@@ -533,4 +549,5 @@
         <state_interface name="Present Velocity"/>
         <state_interface name="Present Current"/>
+        <state_interface name="Error Code"/>
         <param name="Drive Mode">4</param>
         <param name="Operating Mode">3</param>
@@ -556,4 +573,5 @@
         <state_interface name="Present Velocity"/>
         <state_interface name="Present Current"/>
+        <state_interface name="Hardware Error Status"/>
         <param name="Drive Mode">5</param>
         <param name="Operating Mode">3</param>
@@ -576,4 +594,5 @@
         <state_interface name="Present Velocity"/>
         <state_interface name="Present Current"/>
+        <state_interface name="Hardware Error Status"/>
         <param name="Drive Mode">4</param>
         <param name="Operating Mode">3</param>

File: ffw_description/ros2_control/ffw_bg2_rev4_follower/ffw_bg2_follower.ros2_control.xacro (robot description, xacro)
@@ -195,4 +195,5 @@
         <state_interface name="Present Velocity"/>
         <state_interface name="Present Current"/>
+        <state_interface name="Error Code"/>
         <param name="Drive Mode">5</param>
         <param name="Operating Mode">3</param>
@@ -218,4 +219,5 @@
         <state_interface name="Present Velocity"/>
         <state_interface name="Present Current"/>
+        <state_interface name="Error Code"/>
         <param name="Drive Mode">4</param>
         <param name="Operating Mode">3</param>
@@ -241,4 +243,5 @@
         <state_interface name="Present Velocity"/>
         <state_interface name="Present Current"/>
+        <state_interface name="Error Code"/>
         <param name="Drive Mode">5</param>
         <param name="Operating Mode">3</param>
@@ -264,4 +267,5 @@
         <state_interface name="Present Velocity"/>
         <state_interface name="Present Current"/>
+        <state_interface name="Error Code"/>
         <param name="Drive Mode">5</param>
         <param name="Operating Mode">3</param>
@@ -287,4 +291,5 @@
         <state_interface name="Present Velocity"/>
         <state_interface name="Present Current"/>
+        <state_interface name="Error Code"/>
         <param name="Drive Mode">5</param>
         <param name="Operating Mode">3</param>
@@ -310,4 +315,5 @@
         <state_interface name="Present Velocity"/>
         <state_interface name="Present Current"/>
+        <state_interface name="Error Code"/>
         <param name="Drive Mode">5</param>
         <param name="Operating Mode">3</param>
@@ -333,4 +339,5 @@
         <state_interface name="Present Velocity"/>
         <state_interface name="Present Current"/>
+        <state_interface name="Hardware Error Status"/>
         <param name="Drive Mode">4</param>
         <param name="Operating Mode">3</param>
@@ -351,4 +358,5 @@
         <state_interface name="Present Velocity"/>
         <state_interface name="Present Current"/>
+        <state_interface name="Hardware Error Status"/>
         <param name="Operating Mode">5</param>
         <param name="Return Delay Time">0</param>
@@ -364,4 +372,5 @@
         <state_interface name="Present Velocity"/>
         <state_interface name="Present Current"/>
+        <state_interface name="Error Code"/>
         <param name="Drive Mode">4</param>
         <param name="Operating Mode">3</param>
@@ -387,4 +396,5 @@
         <state_interface name="Present Velocity"/>
         <state_interface name="Present Current"/>
+        <state_interface name="Error Code"/>
         <param name="Drive Mode">4</param>
         <param name="Operating Mode">3</param>
@@ -410,4 +420,5 @@
         <state_interface name="Present Velocity"/>
         <state_interface name="Present Current"/>
+        <state_interface name="Error Code"/>
         <param name="Drive Mode">5</param>
         <param name="Operating Mode">3</param>
@@ -433,4 +444,5 @@
         <state_interface name="Present Velocity"/>
         <state_interface name="Present Current"/>
+        <state_interface name="Error Code"/>
         <param name="Drive Mode">4</param>
         <param name="Operating Mode">3</param>
@@ -456,4 +468,5 @@
         <state_interface name="Present Velocity"/>
         <state_interface name="Present Current"/>
+        <state_interface name="Error Code"/>
         <param name="Drive Mode">5</param>
         <param name="Operating Mode">3</param>
@@ -479,4 +492,5 @@
         <state_interface name="Present Velocity"/>
         <state_interface name="Present Current"/>
+        <state_interface name="Error Code"/>
         <param name="Drive Mode">4</param>
         <param name="Operating Mode">3</param>
@@ -502,4 +516,5 @@
         <state_interface name="Present Velocity"/>
         <state_interface name="Present Current"/>
+        <state_interface name="Hardware Error Status"/>
         <param name="Drive Mode">4</param>
         <param name="Operating Mode">3</param>
@@ -520,4 +535,5 @@
         <state_interface name="Present Velocity"/>
         <state_interface name="Present Current"/>
+        <state_interface name="Hardware Error Status"/>
         <param name="Operating Mode">5</param>
         <param name="Return Delay Time">0</param>
@@ -533,4 +549,5 @@
         <state_interface name="Present Velocity"/>
         <state_interface name="Present Current"/>
+        <state_interface name="Error Code"/>
         <param name="Drive Mode">4</param>
         <param name="Operating Mode">3</param>
@@ -556,4 +573,5 @@
         <state_interface name="Present Velocity"/>
         <state_interface name="Present Current"/>
+        <state_interface name="Hardware Error Status"/>
         <param name="Drive Mode">5</param>
         <param name="Operating Mode">3</param>
@@ -576,4 +594,5 @@
         <state_interface name="Present Velocity"/>
         <state_interface name="Present Current"/>
+        <state_interface name="Hardware Error Status"/>
         <param name="Drive Mode">5</param>
         <param name="Operating Mode">3</param>

File: ffw_description/ros2_control/ffw_sg2_rev1_follower/ffw_sg2_base.ros2_control.xacro (robot description, xacro)
@@ -33,8 +33,8 @@
               0, 0, 1
             </param>
-            <param name="dynamixel_state_pub_msg_name">dynamixel_hardware_interface/dxl_state</param>
-            <param name="get_dynamixel_data_srv_name">dynamixel_hardware_interface/get_dxl_data</param>
-            <param name="set_dynamixel_data_srv_name">dynamixel_hardware_interface/set_dxl_data</param>
-            <param name="reboot_dxl_srv_name">dynamixel_hardware_interface/reboot_dxl</param>
+            <param name="dynamixel_state_pub_msg_name">ffw_base/dxl_state</param>
+            <param name="get_dynamixel_data_srv_name">ffw_base/get_dxl_data</param>
+            <param name="set_dynamixel_data_srv_name">ffw_base/set_dxl_data</param>
+            <param name="reboot_dxl_srv_name">ffw_base/reboot_dxl</param>
             <param name="set_dxl_torque_srv_name">dynamixel_hardware_interface/set_dxl_torque</param>
             <param name="error_timeout_ms">500</param>

File: ffw_description/ros2_control/ffw_sg2_rev1_follower/ffw_sg2_follower.ros2_control.xacro (robot description, xacro)
@@ -71,8 +71,8 @@
               0, 0, 0, 0, 0, 0, 0, 0, 0, 0, 0, 0, 0, 0, 0, 0, 0, 0, 0, 0, 0, 1
             </param>
-            <param name="dynamixel_state_pub_msg_name">dynamixel_hardware_interface/dxl_state</param>
-            <param name="get_dynamixel_data_srv_name">dynamixel_hardware_interface/get_dxl_data</param>
-            <param name="set_dynamixel_data_srv_name">dynamixel_hardware_interface/set_dxl_data</param>
-            <param name="reboot_dxl_srv_name">dynamixel_hardware_interface/reboot_dxl</param>
+            <param name="dynamixel_state_pub_msg_name">ffw_follower/dxl_state</param>
+            <param name="get_dynamixel_data_srv_name">ffw_follower/get_dxl_data</param>
+            <param name="set_dynamixel_data_srv_name">ffw_follower/set_dxl_data</param>
+            <param name="reboot_dxl_srv_name">ffw_follower/reboot_dxl</param>
             <param name="set_dxl_torque_srv_name">dynamixel_hardware_interface/set_dxl_torque</param>
           </xacro:unless>
@@ -219,4 +219,5 @@
         <state_interface name="Present Velocity"/>
         <state_interface name="Present Current"/>
+        <state_interface name="Error Code"/>
         <param name="Drive Mode">5</param>
         <param name="Operating Mode">3</param>
@@ -242,4 +243,5 @@
         <state_interface name="Present Velocity"/>
         <state_interface name="Present Current"/>
+        <state_interface name="Error Code"/>
         <param name="Drive Mode">4</param>
         <param name="Operating Mode">3</param>
@@ -265,4 +267,5 @@
         <state_interface name="Present Velocity"/>
         <state_interface name="Present Current"/>
+        <state_interface name="Error Code"/>
         <param name="Drive Mode">5</param>
         <param name="Operating Mode">3</param>
@@ -288,4 +291,5 @@
         <state_interface name="Present Velocity"/>
         <state_interface name="Present Current"/>
+        <state_interface name="Error Code"/>
         <param name="Drive Mode">5</param>
         <param name="Operating Mode">3</param>
@@ -311,4 +315,5 @@
         <state_interface name="Present Velocity"/>
         <state_interface name="Present Current"/>
+        <state_interface name="Error Code"/>
         <param name="Drive Mode">5</param>
         <param name="Operating Mode">3</param>
@@ -334,4 +339,5 @@
         <state_interface name="Present Velocity"/>
         <state_interface name="Present Current"/>
+        <state_interface name="Error Code"/>
         <param name="Drive Mode">5</param>
         <param name="Operating Mode">3</param>
@@ -357,4 +363,5 @@
         <state_interface name="Present Velocity"/>
         <state_interface name="Present Current"/>
+        <state_interface name="Hardware Error Status"/>
         <param name="Drive Mode">4</param>
         <param name="Operating Mode">3</param>
@@ -375,4 +382,5 @@
         <state_interface name="Present Velocity"/>
         <state_interface name="Present Current"/>
+        <state_interface name="Hardware Error Status"/>
         <param name="Operating Mode">5</param>
         <param name="Return Delay Time">0</param>
@@ -388,4 +396,5 @@
         <state_interface name="Present Velocity"/>
         <state_interface name="Present Current"/>
+        <state_interface name="Error Code"/>
         <param name="Drive Mode">4</param>
         <param name="Operating Mode">3</param>
@@ -411,4 +420,5 @@
         <state_interface name="Present Velocity"/>
         <state_interface name="Present Current"/>
+        <state_interface name="Error Code"/>
         <param name="Drive Mode">4</param>
         <param name="Operating Mode">3</param>
@@ -434,4 +444,5 @@
         <state_interface name="Present Velocity"/>
         <state_interface name="Present Current"/>
+        <state_interface name="Error Code"/>
         <param name="Drive Mode">5</param>
         <param name="Operating Mode">3</param>
@@ -457,4 +468,5 @@
         <state_interface name="Present Velocity"/>
         <state_interface name="Present Current"/>
+        <state_interface name="Error Code"/>
         <param name="Drive Mode">4</param>
         <param name="Operating Mode">3</param>
@@ -480,4 +492,5 @@
         <state_interface name="Present Velocity"/>
         <state_interface name="Present Current"/>
+        <state_interface name="Error Code"/>
         <param name="Drive Mode">5</param>
         <param name="Operating Mode">3</param>
@@ -503,4 +516,5 @@
         <state_interface name="Present Velocity"/>
         <state_interface name="Present Current"/>
+        <state_interface name="Error Code"/>
         <param name="Drive Mode">4</param>
         <param name="Operating Mode">3</param>
@@ -526,4 +540,5 @@
         <state_interface name="Present Velocity"/>
         <state_interface name="Present Current"/>
+        <state_interface name="Hardware Error Status"/>
         <param name="Drive Mode">4</param>
         <param name="Operating Mode">3</param>
@@ -544,4 +559,5 @@
         <state_interface name="Present Velocity"/>
         <state_interface name="Present Current"/>
+        <state_interface name="Hardware Error Status"/>
         <param name="Operating Mode">5</param>
         <param name="Return Delay Time">0</param>
@@ -557,4 +573,5 @@
         <state_interface name="Present Velocity"/>
         <state_interface name="Present Current"/>
+        <state_interface name="Error Code"/>
         <param name="Drive Mode">4</param>
         <param name="Operating Mode">3</param>
@@ -580,4 +597,5 @@
         <state_interface name="Present Velocity"/>
         <state_interface name="Present Current"/>
+        <state_interface name="Hardware Error Status"/>
         <param name="Drive Mode">5</param>
         <param name="Operating Mode">3</param>
@@ -600,4 +618,5 @@
         <state_interface name="Present Velocity"/>
         <state_interface name="Present Current"/>
+        <state_interface name="Hardware Error Status"/>
         <param name="Drive Mode">5</param>
         <param name="Operating Mode">3</param>
@@ -621,4 +640,5 @@
         <state_interface name="Present Velocity"/>
         <state_interface name="Present Current"/>
+        <state_interface name="Error Code"/>
         <param name="Drive Mode">5</param>
         <param name="Operating Mode">3</param>
@@ -641,4 +661,5 @@
         <state_interface name="Present Velocity"/>
         <state_interface name="Present Current"/>
+        <state_interface name="Error Code"/>
         <param name="Drive Mode">5</param>
         <param name="Operating Mode">3</param>
@@ -661,4 +682,5 @@
         <state_interface name="Present Velocity"/>
         <state_interface name="Present Current"/>
+        <state_interface name="Error Code"/>
         <param name="Drive Mode">5</param>
         <param name="Operating Mode">3</param>

File: ffw_description/ros2_control/ffw_sg2_rev1_follower/ffw_sg2_sensor.ros2_control.xacro (robot description, xacro)
@@ -21,9 +21,9 @@
             <param name="transmission_to_joint_matrix"></param>
             <param name="joint_to_transmission_matrix"></param>
-            <param name="dynamixel_state_pub_msg_name">dynamixel_hardware_interface/dxl_state</param>
-            <param name="get_dynamixel_data_srv_name">dynamixel_hardware_interface/get_dxl_data</param>
-            <param name="set_dynamixel_data_srv_name">dynamixel_hardware_interface/set_dxl_data</param>
-            <param name="reboot_dxl_srv_name">dynamixel_hardware_interface/reboot_dxl</param>
-            <param name="set_dxl_torque_srv_name">dynamixel_hardware_interface/set_dxl_torque</param>
+            <param name="dynamixel_state_pub_msg_name">ffw_sensor/dxl_state</param>
+            <param name="get_dynamixel_data_srv_name">ffw_sensor/get_dxl_data</param>
+            <param name="set_dynamixel_data_srv_name">ffw_sensor/set_dxl_data</param>
+            <param name="reboot_dxl_srv_name">ffw_sensor/reboot_dxl</param>
+            <param name="set_dxl_torque_srv_name">ffw_sensor/set_dxl_torque</param>
           </xacro:unless>
         </hardware>

File: ffw_description/urdf/ffw_sg2_rev1_follower/ffw_sg2_follower.urdf.xacro (robot description, xacro)
@@ -13,10 +13,4 @@
   <xacro:include filename="$(find ffw_description)/ros2_control/$(arg model)/ffw_sg2_sensor.ros2_control.xacro" />
   <xacro:include filename="$(find ffw_description)/gazebo/$(arg model)/ffw_sg2_follower.gazebo.xacro" />
-  <link name="world"/>
-  <joint name="$(arg prefix)world_fixed" type="fixed">
-    <parent link="world"/>
-    <child link="$(arg prefix)base_link"/>
-    <origin xyz="0.0 0.0 0.0" rpy="0 0 0"/>
-  </joint>
   <link name="$(arg prefix)base_link">
     <visual>
@@ -86,5 +80,5 @@
       <origin xyz="0.1371 0.2554 0.27555" rpy="0 0 0"/>
       <axis xyz="0 0 1" />
-      <limit velocity="4.8" effort="1" lower="${-pi*6.0}" upper="${pi*6.0}" />
+      <limit velocity="9999.0" effort="9999.0" lower="${-pi*6.0}" upper="${pi*6.0}" />
   </joint>
   <link name="$(arg prefix)left_wheel_steer_link">
@@ -112,10 +106,10 @@
     </inertial>
   </link>
-  <joint name="$(arg prefix)left_wheel_drive" type="revolute">
+  <joint name="$(arg prefix)left_wheel_drive" type="continuous">
       <parent link="$(arg prefix)left_wheel_steer_link"/>
       <child link="$(arg prefix)left_wheel_drive_link"/>
       <origin xyz="0 0 -0.18905" rpy="0 0 0"/>
       <axis xyz="0 1 0" />
-      <limit velocity="4.8" effort="1" lower="${-pi*6.0}" upper="${pi*6.0}" />
+      <limit velocity="9999.0" effort="9999.0"/>
   </joint>
   <link name="$(arg prefix)left_wheel_drive_link">
@@ -148,5 +142,5 @@
       <origin xyz="0.1371 -0.2554 0.27555" rpy="0 0 0"/>
       <axis xyz="0 0 1" />
-      <limit velocity="4.8" effort="1" lower="${-pi*6.0}" upper="${pi*6.0}" />
+      <limit velocity="9999.0" effort="9999.0" lower="${-pi*6.0}" upper="${pi*6.0}" />
   </joint>
   <link name="$(arg prefix)right_wheel_steer_link">
@@ -174,10 +168,10 @@
     </inertial>
   </link>
-  <joint name="$(arg prefix)right_wheel_drive" type="revolute">
+  <joint name="$(arg prefix)right_wheel_drive" type="continuous">
       <parent link="$(arg prefix)right_wheel_steer_link"/>
       <child link="$(arg prefix)right_wheel_drive_link"/>
       <origin xyz="0 0 -0.18905" rpy="0 0 0"/>
       <axis xyz="0 1 0" />
-      <limit velocity="4.8" effort="1" lower="${-pi*6.0}" upper="${pi*6.0}" />
+      <limit velocity="9999.0" effort="9999.0"/>
   </joint>
   <link name="$(arg prefix)right_wheel_drive_link">
@@ -210,5 +204,5 @@
       <origin xyz="-0.2899 0 0.27555" rpy="0 0 0"/>
       <axis xyz="0 0 1" />
-      <limit velocity="4.8" effort="1" lower="${-pi*6.0}" upper="${pi*6.0}" />
+      <limit velocity="9999.0" effort="9999.0" lower="${-pi*6.0}" upper="${pi*6.0}" />
   </joint>
   <link name="$(arg prefix)rear_wheel_steer_link">
@@ -236,10 +230,10 @@
     </inertial>
   </link>
-  <joint name="$(arg prefix)rear_wheel_drive" type="revolute">
+  <joint name="$(arg prefix)rear_wheel_drive" type="continuous">
       <parent link="$(arg prefix)rear_wheel_steer_link"/>
       <child link="$(arg prefix)rear_wheel_drive_link"/>
       <origin xyz="0 0 -0.18905" rpy="0 0 0"/>
       <axis xyz="0 1 0" />
-      <limit velocity="4.8" effort="1" lower="${-pi*6.0}" upper="${pi*6.0}" />
+      <limit velocity="9999.0" effort="9999.0"/>
   </joint>
   <link name="$(arg prefix)rear_wheel_drive_link">
